File: pcb/power-supply.kicad_sch (KiCad schematic)
At the start: 11 parts, among them J1 AMT0440007DB0000G, J2 AMT0440007DB0000G, J3 AMT0440007DB0000G, J4 AMT0440007DB0000G, U9 NCP718BSNADJT1G

Commit message: Move symbols and footprints to single common lib
Having a unique library for each component makes the components
difficult to search. Moving them under a single library, `lib`, makes
them easier to find.
Parts:
- J1, J2, J3, J4: footprint CONN_AMT0440007DB0000G_AMP -> lib:CONN_AMT0440007DB0000G_AMP; symbol AMT0440007DB0000G:AMT0440007DB0000G -> lib:AMT0440007DB0000G; DigiKey Part Number 732-74650074RCT-ND -> 1818-AMT0440007DB0000G-ND; DigiKey URL https://www.digikey.com/en/products/detail/w%C3%BCrth-elekt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 -> https://www.digikey.com/en/products/detail/amphenol-anytek/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
Changed lines of the file:
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@@
 	)
 	(symbol
-		(lib_id "AMT0440007DB0000G:AMT0440007DB0000G")
+		(lib_id "lib:AMT0440007DB0000G")
 		(at 99.06 102.87 270)
 		(unit 1)
@@
 			)
 		)
-		(property "Footprint" "CONN_AMT0440007DB0000G_AMP"
+		(property "Footprint" "lib:CONN_AMT0440007DB0000G_AMP"
 			(at 99.06 102.87 0)
 			(hide yes)
@@
 			)
 		)
-		(property "Datasheet" "AMT0440007DB0000G"
+		(property "Datasheet" "kicad-embed://AMT0440007DB0000G.pdf"
 			(at 99.06 102.87 0)
 			(hide yes)
@@
 			)
 		)
-		(property "Description" "6 Pin Screw Terminal, Power Tap M8 Through Hole"
+		(property "Description" "Screw Terminal"
 			(at 99.06 102.87 0)
 			(hide yes)
@@
 			)
 		)
-		(property "DigiKey Part Number" "732-74650074RCT-ND"
+		(property "DigiKey Part Number" "1818-AMT0440007DB0000G-ND"
 			(at 99.06 102.87 0)
 			(hide yes)
@@
 			)
 		)
-		(property "DigiKey URL" "https://www.digikey.com/en/products/detail/w%C3%BCrth-elektronik/74650074R/6643979"
+		(property "DigiKey URL" "https://www.digikey.com/en/products/detail/amphenol-anytek/AMT0440007DB0000G/21777826"
 			(at 99.06 102.87 0)
 			(hide yes)
@@
 	)
 	(symbol
-		(lib_name "AMT0440007DB0000G_1")
-		(lib_id "AMT0440007DB0000G:AMT0440007DB0000G")
+		(lib_id "lib:AMT0440007DB0000G")
 		(at 76.2 87.63 90)
 		(unit 1)
@@
 			)
 		)
-		(property "Footprint" "CONN_AMT0440007DB0000G_AMP"
+		(property "Footprint" "lib:CONN_AMT0440007DB0000G_AMP"
 			(at 76.2 87.63 0)
 			(hide yes)
@@
 			)
 		)
-		(property "Datasheet" "AMT0440007DB0000G"
+		(property "Datasheet" "kicad-embed://AMT0440007DB0000G.pdf"
 			(at 76.2 87.63 0)
 			(hide yes)
@@
 			)
 		)
-		(property "Description" "6 Pin Screw Terminal, Power Tap M8 Through Hole"
+		(property "Description" "Screw Terminal"
 			(at 76.2 87.63 0)
 			(hide yes)
@@
 			)
 		)
-		(property "DigiKey Part Number" "732-74650074RCT-ND"
+		(property "DigiKey Part Number" "1818-AMT0440007DB0000G-ND"
 			(at 76.2 87.63 0)
 			(hide yes)
@@
 			)
 		)
-		(property "DigiKey URL" "https://www.digikey.com/en/products/detail/w%C3%BCrth-elektronik/74650074R/6643979"
+		(property "DigiKey URL" "https://www.digikey.com/en/products/detail/amphenol-anytek/AMT0440007DB0000G/21777826"
 			(at 76.2 87.63 0)
 			(hide yes)
@@
 	)
 	(symbol
-		(lib_name "AMT0440007DB0000G_2")
-		(lib_id "AMT0440007DB0000G:AMT0440007DB0000G")
+		(lib_id "lib:AMT0440007DB0000G")
 		(at 91.44 87.63 90)
 		(unit 1)
@@
 			)
 		)
-		(property "Footprint" "CONN_AMT0440007DB0000G_AMP"
+		(property "Footprint" "lib:CONN_AMT0440007DB0000G_AMP"
 			(at 91.44 87.63 0)
 			(hide yes)
@@
 			)
 		)
-		(property "Datasheet" "AMT0440007DB0000G"
+		(property "Datasheet" "kicad-embed://AMT0440007DB0000G.pdf"
 			(at 91.44 87.63 0)
 			(hide yes)
@@
 			)
 		)
-		(property "Description" "6 Pin Screw Terminal, Power Tap M8 Through Hole"
+		(property "Description" "Screw Terminal"
 			(at 91.44 87.63 0)
 			(hide yes)
@@
 			)
 		)
-		(property "DigiKey Part Number" "732-74650074RCT-ND"
+		(property "DigiKey Part Number" "1818-AMT0440007DB0000G-ND"
 			(at 91.44 87.63 0)
 			(hide yes)
@@
 			)
 		)
-		(property "DigiKey URL" "https://www.digikey.com/en/products/detail/w%C3%BCrth-elektronik/74650074R/6643979"
+		(property "DigiKey URL" "https://www.digikey.com/en/products/detail/amphenol-anytek/AMT0440007DB0000G/21777826"
 			(at 91.44 87.63 0)
 			(hide yes)
@@
 	)
 	(symbol
-		(lib_name "AMT0440007DB0000G_3")
-		(lib_id "AMT0440007DB0000G:AMT0440007DB0000G")
+		(lib_id "lib:AMT0440007DB0000G")
 		(at 83.82 102.87 270)
 		(unit 1)
@@
 			)
 		)
-		(property "Footprint" "CONN_AMT0440007DB0000G_AMP"
+		(property "Footprint" "lib:CONN_AMT0440007DB0000G_AMP"
 			(at 83.82 102.87 0)
 			(hide yes)
@@
 			)
 		)
-		(property "Datasheet" "AMT0440007DB0000G"
+		(property "Datasheet" "kicad-embed://AMT0440007DB0000G.pdf"
 			(at 83.82 102.87 0)
 			(hide yes)
@@
 			)
 		)
-		(property "Description" "6 Pin Screw Terminal, Power Tap M8 Through Hole"
+		(property "Description" "Screw Terminal"
 			(at 83.82 102.87 0)
 			(hide yes)
@@
 			)
 		)
-		(property "DigiKey Part Number" "732-74650074RCT-ND"
+		(property "DigiKey Part Number" "1818-AMT0440007DB0000G-ND"
 			(at 83.82 102.87 0)
 			(hide yes)
@@
 			)
 		)
-		(property "DigiKey URL" "https://www.digikey.com/en/products/detail/w%C3%BCrth-elektronik/74650074R/6643979"
+		(property "DigiKey URL" "https://www.digikey.com/en/products/detail/amphenol-anytek/AMT0440007DB0000G/21777826"
 			(at 83.82 102.87 0)
 			(hide yes)

Commit message: Assign footprints for components
Parts:
- C1, C7, C8: footprint (none) -> Capacitor_SMD:C_0805_2012Metric_Pad1.18x1.45mm_HandSolder
- JP3: footprint (none) -> Connector_PinHeader_2.54mm:PinHeader_1x03_P2.54mm_Vertical
- R6, R7: footprint (none) -> Resistor_SMD:R_0805_2012Metric_Pad1.20x1.40mm_HandSolder
- U9: footprint (none) -> Package_TO_SOT_SMD:TSOT-23-5_HandSoldering
Changed lines of the file:
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@@
 			)
 		)
-		(property "Footprint" ""
+		(property "Footprint" "Package_TO_SOT_SMD:TSOT-23-5_HandSoldering"
 			(at 182.88 96.52 0)
 			(hide yes)
@@
 			)
 		)
-		(property "Footprint" ""
+		(property "Footprint" "Connector_PinHeader_2.54mm:PinHeader_1x03_P2.54mm_Vertical"
 			(at 167.64 97.79 0)
 			(hide yes)
@@
 			)
 		)
-		(property "Footprint" ""
+		(property "Footprint" "Resistor_SMD:R_0805_2012Metric_Pad1.20x1.40mm_HandSolder"
 			(at 195.58 93.98 0)
 			(hide yes)
@@
 	)
 	(symbol
+		(lib_name "AMT0440007DB0000G_1")
 		(lib_id "lib:AMT0440007DB0000G")
 		(at 76.2 87.63 90)
@@
 			)
 		)
-		(property "Footprint" ""
+		(property "Footprint" "Capacitor_SMD:C_0805_2012Metric_Pad1.18x1.45mm_HandSolder"
 			(at 104.14 95.25 0)
 			(hide yes)
@@
 			)
 		)
-		(property "Footprint" ""
+		(property "Footprint" "Capacitor_SMD:C_0805_2012Metric_Pad1.18x1.45mm_HandSolder"
 			(at 146.05 93.98 0)
 			(hide yes)
@@
 	)
 	(symbol
+		(lib_name "AMT0440007DB0000G_2")
 		(lib_id "lib:AMT0440007DB0000G")
 		(at 91.44 87.63 90)
@@
 	)
 	(symbol
+		(lib_name "AMT0440007DB0000G_3")
 		(lib_id "lib:AMT0440007DB0000G")
 		(at 83.82 102.87 270)
@@
 			)
 		)
-		(property "Footprint" ""
+		(property "Footprint" "Capacitor_SMD:C_0805_2012Metric_Pad1.18x1.45mm_HandSolder"
 			(at 208.28 99.06 0)
 			(hide yes)
@@
 			)
 		)
-		(property "Footprint" ""
+		(property "Footprint" "Resistor_SMD:R_0805_2012Metric_Pad1.20x1.40mm_HandSolder"
 			(at 195.58 102.87 0)
 			(hide yes)

Commit message: Add power supply remote control header and labels
Parts:
- JP3: now in the parts list
Changed lines of the file:
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@@
+	(wire
+		(pts
+			(xy 104.14 100.33) (xy 104.14 102.87)
+		)
+		(stroke
+			(width 0)
+			(type default)
+		)
+	)
 	(wire
 		(pts
 			(xy 83.82 90.17) (xy 91.44 90.17)
-		)
-		(stroke
-			(width 0)
-			(type default)
-		)
-	)
-	(wire
-		(pts
-			(xy 104.14 100.33) (xy 104.14 102.87)
 		)
 		(stroke
@@
 		(body_style 1)
 		(exclude_from_sim no)
-		(in_bom no)
+		(in_bom yes)
 		(on_board yes)
 		(in_pos_files yes)

Commit message: Change C1 to be THT electrolytic instead of SMT
C1 is the largest filtering capacitor, which is used for the power
supply. It was previously an 0805 surface mount footprint. Changing it
to a through hole footprint gives us more flexibility if we need a
diferent capacitance.
Parts:
- C1: footprint Capacitor_SMD:C_0805_2012Metric_Pad1.18x1.45mm_HandSolder -> Capacitor_THT:C_Radial_D6.3mm_H11.0mm_P2.50mm
Changed lines of the file:
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@@
 			)
 		)
-		(property "Footprint" "Capacitor_SMD:C_0805_2012Metric_Pad1.18x1.45mm_HandSolder"
+		(property "Footprint" "Capacitor_THT:C_Radial_D6.3mm_H11.0mm_P2.50mm"
 			(at 104.14 95.25 0)
 			(hide yes)
